File: NTPclock/clock.sch (EAGLE design)
At the start: 27 parts, among them IC1 MAX7219CNG

Commit message: organize schematic more
Parts:
- renumbered SG1 to BUZ1
Other:
- moved on the sheet: BAR_GRAPHA, BAR_GRAPHB, BAR_GRAPHC, BAR_GRAPHD, BAR_GRAPHE, BAR_GRAPHF, BAR_GRAPHG, BAR_GRAPHH, BAR_GRAPHI, BAR_GRAPHJ, C3, C4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

Commit message: Silkscreen Labeling improvements
Parts:
- NODEMCU.V3: value NODEMCU V3 -> ESP12E_DEVKIT
- renumbered U$1 to NODEMCU.V3
Changed lines of the file:
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@@
 </classes>
 <parts>
-<part name="U$1" library="NODEMCUv1" deviceset="ESP12E_DEVKIT" device="" value="NODEMCU V3"/>
+<part name="NODEMCU.V3" library="NODEMCUv1" deviceset="ESP12E_DEVKIT" device="" value=""/>
 <part name="IC1" library="max7219" deviceset="MAX7219CNG" device=""/>
 <part name="R1" library="SparkFun-Resistors" deviceset="RESISTOR" device="1206"/>
@@
 </plain>
 <instances>
-<instance part="U$1" gate="G$1" x="218.44" y="104.14"/>
+<instance part="NODEMCU.V3" gate="G$1" x="218.44" y="104.14"/>
 <instance part="IC1" gate="G$1" x="76.2" y="83.82"/>
 <instance part="R1" gate="G$1" x="50.8" y="81.28"/>
@@
 <net name="GND" class="0">
 <segment>
-<pinref part="U$1" gate="G$1" pin="GND@5"/>
+<pinref part="NODEMCU.V3" gate="G$1" pin="GND@5"/>
 <wire x1="200.66" y1="119.38" x2="193.04" y2="119.38" width="0.1524" layer="91"/>
 <wire x1="193.04" y1="119.38" x2="193.04" y2="99.06" width="0.1524" layer="91"/>
-<pinref part="U$1" gate="G$1" pin="GND@1"/>
+<pinref part="NODEMCU.V3" gate="G$1" pin="GND@1"/>
 <wire x1="193.04" y1="99.06" x2="193.04" y2="88.9" width="0.1524" layer="91"/>
 <wire x1="193.04" y1="88.9" x2="200.66" y2="88.9" width="0.1524" layer="91"/>
-<pinref part="U$1" gate="G$1" pin="GND@0"/>
+<pinref part="NODEMCU.V3" gate="G$1" pin="GND@0"/>
 <wire x1="200.66" y1="99.06" x2="193.04" y2="99.06" width="0.1524" layer="91"/>
 <junction x="193.04" y="99.06"/>
 <wire x1="193.04" y1="88.9" x2="193.04" y2="73.66" width="0.1524" layer="91"/>
 <junction x="193.04" y="88.9"/>
-<pinref part="U$1" gate="G$1" pin="GND@3"/>
+<pinref part="NODEMCU.V3" gate="G$1" pin="GND@3"/>
 <wire x1="236.22" y1="88.9" x2="246.38" y2="88.9" width="0.1524" layer="91"/>
 <wire x1="246.38" y1="88.9" x2="246.38" y2="106.68" width="0.1524" layer="91"/>
-<pinref part="U$1" gate="G$1" pin="GND@2"/>
+<pinref part="NODEMCU.V3" gate="G$1" pin="GND@2"/>
 <wire x1="246.38" y1="106.68" x2="236.22" y2="106.68" width="0.1524" layer="91"/>
 <wire x1="246.38" y1="73.66" x2="246.38" y2="88.9" width="0.1524" layer="91"/>
@@
 </segment>
 <segment>
-<pinref part="U$1" gate="G$1" pin="D1"/>
+<pinref part="NODEMCU.V3" gate="G$1" pin="D1"/>
 <wire x1="236.22" y1="119.38" x2="243.84" y2="119.38" width="0.1524" layer="91"/>
 <label x="238.76" y="119.38" size="1.778" layer="95"/>
@@
 </segment>
 <segment>
-<pinref part="U$1" gate="G$1" pin="D2"/>
+<pinref part="NODEMCU.V3" gate="G$1" pin="D2"/>
 <wire x1="236.22" y1="116.84" x2="243.84" y2="116.84" width="0.1524" layer="91"/>
 <label x="238.76" y="116.84" size="1.778" layer="95"/>
@@
 <net name="DATA" class="0">
 <segment>
-<pinref part="U$1" gate="G$1" pin="D5"/>
+<pinref part="NODEMCU.V3" gate="G$1" pin="D5"/>
 <wire x1="236.22" y1="104.14" x2="243.84" y2="104.14" width="0.1524" layer="91"/>
 <label x="238.76" y="104.14" size="1.778" layer="95"/>
@@
 </segment>
 <segment>
-<pinref part="U$1" gate="G$1" pin="D7"/>
+<pinref part="NODEMCU.V3" gate="G$1" pin="D7"/>
 <wire x1="236.22" y1="99.06" x2="243.84" y2="99.06" width="0.1524" layer="91"/>
 <label x="238.76" y="99.06" size="1.778" layer="95"/>
@@
 </segment>
 <segment>
-<pinref part="U$1" gate="G$1" pin="D6"/>
+<pinref part="NODEMCU.V3" gate="G$1" pin="D6"/>
 <wire x1="236.22" y1="101.6" x2="243.84" y2="101.6" width="0.1524" layer="91"/>
 <label x="238.76" y="101.6" size="1.778" layer="95"/>
@@
 <pinref part="SUPPLY3" gate="G$1" pin="VCC"/>
 <wire x1="172.72" y1="99.06" x2="172.72" y2="86.36" width="0.1524" layer="91"/>
-<pinref part="U$1" gate="G$1" pin="VIN"/>
+<pinref part="NODEMCU.V3" gate="G$1" pin="VIN"/>
 <pinref part="C7" gate="G$1" pin="+"/>
 <pinref part="C4" gate="G$1" pin="1"/>
@@
 </segment>
 <segment>
-<pinref part="U$1" gate="G$1" pin="3V3@0"/>
+<pinref part="NODEMCU.V3" gate="G$1" pin="3V3@0"/>
 <pinref part="SUPPLY2" gate="G$1" pin="3.3V"/>
 <wire x1="200.66" y1="96.52" x2="185.42" y2="96.52" width="0.1524" layer="91"/>
@@
 </segment>
 <segment>
-<pinref part="U$1" gate="G$1" pin="3V3@1"/>
+<pinref part="NODEMCU.V3" gate="G$1" pin="3V3@1"/>
 <wire x1="236.22" y1="109.22" x2="243.84" y2="109.22" width="0.1524" layer="91"/>
 <label x="238.76" y="109.22" size="1.778" layer="95"/>
 </segment>
 <segment>
-<pinref part="U$1" gate="G$1" pin="3V3@2"/>
+<pinref part="NODEMCU.V3" gate="G$1" pin="3V3@2"/>
 <wire x1="236.22" y1="86.36" x2="243.84" y2="86.36" width="0.1524" layer="91"/>
 <label x="238.76" y="86.36" size="1.778" layer="95"/>
@@
 <net name="D4" class="0">
 <segment>
-<pinref part="U$1" gate="G$1" pin="D4"/>
+<pinref part="NODEMCU.V3" gate="G$1" pin="D4"/>
 <wire x1="236.22" y1="111.76" x2="243.84" y2="111.76" width="0.1524" layer="91"/>
 <label x="238.76" y="111.76" size="1.778" layer="95"/>
@@
 <net name="D8" class="0">
 <segment>
-<pinref part="U$1" gate="G$1" pin="D8"/>
+<pinref part="NODEMCU.V3" gate="G$1" pin="D8"/>
 <wire x1="236.22" y1="96.52" x2="243.84" y2="96.52" width="0.1524" layer="91"/>
 <label x="238.76" y="96.52" size="1.778" layer="95"/>

Commit message: Added Serial Breakout
Parts:
- removed J2: (no value), SparkFun-Connectors:M02PTH
- added J0: (no value), SparkFun-Connectors:M06POLAR
- added SERIAL: (no value), SparkFun-Connectors:M02PTH
- J1: device SparkFun-Connectors:M06POLAR -> SparkFun-Connectors:M02PTH
Connections:
- new net RX: NODEMCU.V3.RX, SERIAL.2
- new net TX: NODEMCU.V3.TX, SERIAL.1
- net 3.3V: now also J0.2; no longer J1.2
- net 32K: now also J0.6; no longer J1.6
- net D8: now also J1.1; no longer J2.1
- net GND: now also J0.1, J1.2; no longer J1.1, J2.2
- net SCL: now also J0.4; no longer J1.4
- net SDA: now also J0.3; no longer J1.3
- net SQL: now also J0.5; no longer J1.5
Other:
- moved on the sheet: BUZ1, R4
Changed lines of the file:
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@@
 <part name="C8" library="SparkFun-Capacitors" deviceset="CAP_POL" device="PTH1" value="10μF"/>
 <part name="POWER" library="SparkFun-Connectors" deviceset="M02" device="JST-PTH-VERT"/>
-<part name="J1" library="SparkFun-Connectors" deviceset="M06" device="POLAR"/>
+<part name="J0" library="SparkFun-Connectors" deviceset="M06" device="POLAR"/>
 <part name="DIG_3" library="custom_display" deviceset="7-SEGMENT-DISPLAY-REAL-1&quot;" device=""/>
 <part name="DIG_2" library="custom_display" deviceset="7-SEGMENT-DISPLAY-REAL-1&quot;" device=""/>
@@
 <part name="D2" library="SparkFun-LED" deviceset="LED" device="3MM"/>
 <part name="BUZ1" library="SparkFun-Electromechanical" deviceset="BUZZER" device="PTH"/>
-<part name="J2" library="SparkFun-Connectors" deviceset="M02" device="PTH"/>
+<part name="J1" library="SparkFun-Connectors" deviceset="M02" device="PTH"/>
 <part name="R4" library="SparkFun-Resistors" deviceset="RESISTOR" device="1206" value="100Ω"/>
 <part name="GND5" library="SparkFun-Aesthetics" deviceset="GND" device=""/>
 <part name="FRAME1" library="SparkFun-Aesthetics" deviceset="FRAME-LETTER" device=""/>
+<part name="SERIAL" library="SparkFun-Connectors" deviceset="M02" device="PTH"/>
 </parts>
 <sheets>
@@
 <instance part="C8" gate="G$1" x="50.8" y="63.5"/>
 <instance part="POWER" gate="G$1" x="33.02" y="-35.56"/>
-<instance part="J1" gate="G$1" x="81.28" y="-35.56"/>
+<instance part="J0" gate="G$1" x="81.28" y="-35.56"/>
 <instance part="DIG_3" gate="G$1" x="231.14" y="17.78"/>
 <instance part="DIG_2" gate="G$1" x="193.04" y="17.78"/>
@@
 <instance part="D1" gate="G$1" x="154.94" y="22.86" rot="R90"/>
 <instance part="D2" gate="G$1" x="154.94" y="12.7" rot="R90"/>
-<instance part="BUZ1" gate="G$1" x="134.62" y="-43.18" rot="R90"/>
-<instance part="J2" gate="G$1" x="144.78" y="-30.48"/>
-<instance part="R4" gate="G$1" x="149.86" y="-40.64"/>
-<instance part="GND5" gate="1" x="142.24" y="-45.72"/>
+<instance part="BUZ1" gate="G$1" x="129.54" y="-43.18" rot="R90"/>
+<instance part="J1" gate="G$1" x="134.62" y="-25.4"/>
+<instance part="R4" gate="G$1" x="144.78" y="-40.64"/>
+<instance part="GND5" gate="1" x="137.16" y="-45.72"/>
 <instance part="FRAME1" gate="G$1" x="25.4" y="-50.8"/>
 <instance part="FRAME1" gate="V" x="172.72" y="-50.8"/>
+<instance part="SERIAL" gate="G$1" x="154.94" y="-25.4"/>
 </instances>
 <busses>
@@
 </segment>
 <segment>
-<pinref part="J1" gate="G$1" pin="1"/>
+<pinref part="J0" gate="G$1" pin="1"/>
 <label x="86.36" y="-40.64" size="1.778" layer="95"/>
 <pinref part="C5" gate="G$1" pin="2"/>
@@
 </segment>
 <segment>
-<pinref part="J2" gate="G$1" pin="2"/>
-<wire x1="152.4" y1="-27.94" x2="160.02" y2="-27.94" width="0.1524" layer="91"/>
-<label x="154.94" y="-27.94" size="1.778" layer="95"/>
+<pinref part="J1" gate="G$1" pin="2"/>
+<wire x1="142.24" y1="-22.86" x2="149.86" y2="-22.86" width="0.1524" layer="91"/>
+<label x="144.78" y="-22.86" size="1.778" layer="95"/>
 </segment>
 <segment>
 <pinref part="BUZ1" gate="G$1" pin="1"/>
-<wire x1="137.16" y1="-43.18" x2="142.24" y2="-43.18" width="0.1524" layer="91"/>
+<wire x1="132.08" y1="-43.18" x2="137.16" y2="-43.18" width="0.1524" layer="91"/>
 <pinref part="GND5" gate="1" pin="GND"/>
 </segment>
@@
 <net name="32K" class="0">
 <segment>
-<pinref part="J1" gate="G$1" pin="6"/>
+<pinref part="J0" gate="G$1" pin="6"/>
 <wire x1="86.36" y1="-27.94" x2="91.44" y2="-27.94" width="0.1524" layer="91"/>
 <label x="86.36" y="-27.94" size="1.778" layer="95"/>
@@
 <net name="SQL" class="0">
 <segment>
-<pinref part="J1" gate="G$1" pin="5"/>
+<pinref part="J0" gate="G$1" pin="5"/>
 <label x="86.36" y="-30.48" size="1.778" layer="95"/>
 <pinref part="R3" gate="G$1" pin="2"/>
@@
 <net name="SCL" class="0">
 <segment>
-<pinref part="J1" gate="G$1" pin="4"/>
+<pinref part="J0" gate="G$1" pin="4"/>
 <wire x1="86.36" y1="-33.02" x2="91.44" y2="-33.02" width="0.1524" layer="91"/>
 <label x="86.36" y="-33.02" size="1.778" layer="95"/>
@@
 <net name="SDA" class="0">
 <segment>
-<pinref part="J1" gate="G$1" pin="3"/>
+<pinref part="J0" gate="G$1" pin="3"/>
 <wire x1="86.36" y1="-35.56" x2="91.44" y2="-35.56" width="0.1524" layer="91"/>
 <label x="86.36" y="-35.56" size="1.778" layer="95"/>
@@
 <net name="3.3V" class="0">
 <segment>
-<pinref part="J1" gate="G$1" pin="2"/>
+<pinref part="J0" gate="G$1" pin="2"/>
 <label x="86.36" y="-38.1" size="1.778" layer="95"/>
 <pinref part="C5" gate="G$1" pin="1"/>
@@
 <segment>
 <pinref part="R4" gate="G$1" pin="2"/>
-<label x="157.48" y="-40.64" size="1.778" layer="95"/>
-<wire x1="154.94" y1="-40.64" x2="160.02" y2="-40.64" width="0.1524" layer="91"/>
+<label x="152.4" y="-40.64" size="1.778" layer="95"/>
+<wire x1="149.86" y1="-40.64" x2="154.94" y2="-40.64" width="0.1524" layer="91"/>
 </segment>
 </net>
@@
 </segment>
 <segment>
-<pinref part="J2" gate="G$1" pin="1"/>
-<wire x1="152.4" y1="-30.48" x2="160.02" y2="-30.48" width="0.1524" layer="91"/>
-<label x="154.94" y="-30.48" size="1.778" layer="95"/>
+<pinref part="J1" gate="G$1" pin="1"/>
+<wire x1="142.24" y1="-25.4" x2="149.86" y2="-25.4" width="0.1524" layer="91"/>
+<label x="144.78" y="-25.4" size="1.778" layer="95"/>
 </segment>
 </net>
@@
 <pinref part="R4" gate="G$1" pin="1"/>
 <pinref part="BUZ1" gate="G$1" pin="2"/>
-<wire x1="144.78" y1="-40.64" x2="137.16" y2="-40.64" width="0.1524" layer="91"/>
-</segment>
-</net>
+<wire x1="139.7" y1="-40.64" x2="132.08" y2="-40.64" width="0.1524" layer="91"/>
+</segment>
+</net>
+<net name="RX" class="0">
+<segment>
+<pinref part="NODEMCU.V3" gate="G$1" pin="RX"/>
+<wire x1="236.22" y1="93.98" x2="243.84" y2="93.98" width="0.1524" layer="91"/>
+<label x="238.76" y="93.98" size="1.778" layer="95"/>
+</segment>
+<segment>
+<pinref part="SERIAL" gate="G$1" pin="2"/>
+<wire x1="162.56" y1="-22.86" x2="170.18" y2="-22.86" width="0.1524" layer="91"/>
+<label x="165.1" y="-22.86" size="1.778" layer="95"/>
+</segment>
+</net>
+<net name="TX" class="0">
+<segment>
+<pinref part="NODEMCU.V3" gate="G$1" pin="TX"/>
+<wire x1="236.22" y1="91.44" x2="243.84" y2="91.44" width="0.1524" layer="91"/>
+<label x="238.76" y="91.44" size="1.778" layer="95"/>
+</segment>
+<segment>
+<pinref part="SERIAL" gate="G$1" pin="1"/>
+<wire x1="162.56" y1="-25.4" x2="170.18" y2="-25.4" width="0.1524" layer="91"/>
+<label x="165.1" y="-25.4" size="1.778" layer="95"/>
+</segment>
+</net>

Commit message: Correct bar graph ordering
Connections:
- net A: now also BAR_GRAPHD.A, BAR_GRAPHI.A; no longer BAR_GRAPHB.A, BAR_GRAPHG.A
- net C: now also BAR_GRAPHB.A, BAR_GRAPHG.A; no longer BAR_GRAPHD.A, BAR_GRAPHI.A
- net D: now also BAR_GRAPHA.A, BAR_GRAPHF.A; no longer BAR_GRAPHE.A, BAR_GRAPHJ.A
- net DP: now also BAR_GRAPHE.A, BAR_GRAPHJ.A; no longer BAR_GRAPHA.A, BAR_GRAPHF.A
Changed lines of the file:
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@@
+</segment>
+<segment>
+<pinref part="BAR_GRAPH" gate="I" pin="A"/>
+<wire x1="248.92" y1="7.62" x2="256.54" y2="7.62" width="0.1524" layer="91"/>
+</segment>
+<segment>
+<pinref part="BAR_GRAPH" gate="D" pin="A"/>
+<wire x1="248.92" y1="22.86" x2="256.54" y2="22.86" width="0.1524" layer="91"/>
+</segment>
+</net>
+<net name="B" class="0">
+<segment>
+<pinref part="DIG_3" gate="G$1" pin="B"/>
+<wire x1="208.28" y1="25.4" x2="210.82" y2="25.4" width="0.1524" layer="91"/>
+</segment>
+<segment>
+<pinref part="DIG_1" gate="G$1" pin="B"/>
+<wire x1="109.22" y1="25.4" x2="111.76" y2="25.4" width="0.1524" layer="91"/>
+</segment>
+<segment>
+<pinref part="DIG_2" gate="G$1" pin="B"/>
+<wire x1="170.18" y1="25.4" x2="172.72" y2="25.4" width="0.1524" layer="91"/>
+</segment>
+<segment>
+<pinref part="DIG_0" gate="G$1" pin="B"/>
+<wire x1="71.12" y1="25.4" x2="73.66" y2="25.4" width="0.1524" layer="91"/>
+</segment>
+<segment>
+<pinref part="IC1" gate="G$1" pin="SEGB"/>
+<wire x1="91.44" y1="78.74" x2="88.9" y2="78.74" width="0.1524" layer="91"/>
+</segment>
+<segment>
+<pinref part="BAR_GRAPH" gate="H" pin="A"/>
+<wire x1="248.92" y1="10.16" x2="256.54" y2="10.16" width="0.1524" layer="91"/>
+</segment>
+<segment>
+<pinref part="BAR_GRAPH" gate="C" pin="A"/>
+<wire x1="248.92" y1="25.4" x2="256.54" y2="25.4" width="0.1524" layer="91"/>
+</segment>
+</net>
+<net name="C" class="0">
+<segment>
+<pinref part="DIG_3" gate="G$1" pin="C"/>
+<wire x1="208.28" y1="22.86" x2="210.82" y2="22.86" width="0.1524" layer="91"/>
+</segment>
+<segment>
+<pinref part="DIG_1" gate="G$1" pin="C"/>
+<wire x1="109.22" y1="22.86" x2="111.76" y2="22.86" width="0.1524" layer="91"/>
+</segment>
+<segment>
+<pinref part="DIG_2" gate="G$1" pin="C"/>
+<wire x1="170.18" y1="22.86" x2="172.72" y2="22.86" width="0.1524" layer="91"/>
+</segment>
+<segment>
+<pinref part="DIG_0" gate="G$1" pin="C"/>
+<wire x1="71.12" y1="22.86" x2="73.66" y2="22.86" width="0.1524" layer="91"/>
+</segment>
+<segment>
+<pinref part="IC1" gate="G$1" pin="SEGC"/>
+<wire x1="91.44" y1="76.2" x2="88.9" y2="76.2" width="0.1524" layer="91"/>
+</segment>
+<segment>
+<pinref part="BAR_GRAPH" gate="G" pin="A"/>
+<wire x1="248.92" y1="12.7" x2="256.54" y2="12.7" width="0.1524" layer="91"/>
 </segment>
 <segment>
@@
 <wire x1="248.92" y1="27.94" x2="256.54" y2="27.94" width="0.1524" layer="91"/>
 </segment>
-<segment>
-<pinref part="BAR_GRAPH" gate="G" pin="A"/>
-<wire x1="248.92" y1="12.7" x2="256.54" y2="12.7" width="0.1524" layer="91"/>
-</segment>
-</net>
-<net name="B" class="0">
-<segment>
-<pinref part="DIG_3" gate="G$1" pin="B"/>
-<wire x1="208.28" y1="25.4" x2="210.82" y2="25.4" width="0.1524" layer="91"/>
-</segment>
-<segment>
-<pinref part="DIG_1" gate="G$1" pin="B"/>
-<wire x1="109.22" y1="25.4" x2="111.76" y2="25.4" width="0.1524" layer="91"/>
-</segment>
-<segment>
-<pinref part="DIG_2" gate="G$1" pin="B"/>
-<wire x1="170.18" y1="25.4" x2="172.72" y2="25.4" width="0.1524" layer="91"/>
-</segment>
-<segment>
-<pinref part="DIG_0" gate="G$1" pin="B"/>
-<wire x1="71.12" y1="25.4" x2="73.66" y2="25.4" width="0.1524" layer="91"/>
-</segment>
-<segment>
-<pinref part="IC1" gate="G$1" pin="SEGB"/>
-<wire x1="91.44" y1="78.74" x2="88.9" y2="78.74" width="0.1524" layer="91"/>
-</segment>
-<segment>
-<pinref part="BAR_GRAPH" gate="C" pin="A"/>
-<wire x1="248.92" y1="25.4" x2="256.54" y2="25.4" width="0.1524" layer="91"/>
-</segment>
-<segment>
-<pinref part="BAR_GRAPH" gate="H" pin="A"/>
-<wire x1="248.92" y1="10.16" x2="256.54" y2="10.16" width="0.1524" layer="91"/>
-</segment>
-</net>
-<net name="C" class="0">
-<segment>
-<pinref part="DIG_3" gate="G$1" pin="C"/>
-<wire x1="208.28" y1="22.86" x2="210.82" y2="22.86" width="0.1524" layer="91"/>
-</segment>
-<segment>
-<pinref part="DIG_1" gate="G$1" pin="C"/>
-<wire x1="109.22" y1="22.86" x2="111.76" y2="22.86" width="0.1524" layer="91"/>
-</segment>
-<segment>
-<pinref part="DIG_2" gate="G$1" pin="C"/>
-<wire x1="170.18" y1="22.86" x2="172.72" y2="22.86" width="0.1524" layer="91"/>
-</segment>
-<segment>
-<pinref part="DIG_0" gate="G$1" pin="C"/>
-<wire x1="71.12" y1="22.86" x2="73.66" y2="22.86" width="0.1524" layer="91"/>
-</segment>
-<segment>
-<pinref part="IC1" gate="G$1" pin="SEGC"/>
-<wire x1="91.44" y1="76.2" x2="88.9" y2="76.2" width="0.1524" layer="91"/>
-</segment>
-<segment>
-<pinref part="BAR_GRAPH" gate="D" pin="A"/>
-<wire x1="248.92" y1="22.86" x2="256.54" y2="22.86" width="0.1524" layer="91"/>
-</segment>
-<segment>
-<pinref part="BAR_GRAPH" gate="I" pin="A"/>
-<wire x1="248.92" y1="7.62" x2="256.54" y2="7.62" width="0.1524" layer="91"/>
-</segment>
 </net>
 <net name="D" class="0">
@@
 <pinref part="IC1" gate="G$1" pin="SEGD"/>
 <wire x1="91.44" y1="73.66" x2="88.9" y2="73.66" width="0.1524" layer="91"/>
-</segment>
-<segment>
-<pinref part="BAR_GRAPH" gate="E" pin="A"/>
-<wire x1="248.92" y1="20.32" x2="256.54" y2="20.32" width="0.1524" layer="91"/>
-</segment>
-<segment>
-<pinref part="BAR_GRAPH" gate="J" pin="A"/>
-<wire x1="248.92" y1="5.08" x2="256.54" y2="5.08" width="0.1524" layer="91"/>
 </segment>
 <segment>
@@
 <wire x1="147.32" y1="35.56" x2="147.32" y2="12.7" width="0.1524" layer="91"/>
 </segment>
+<segment>
+<pinref part="BAR_GRAPH" gate="F" pin="A"/>
+<wire x1="248.92" y1="15.24" x2="256.54" y2="15.24" width="0.1524" layer="91"/>
+</segment>
+<segment>
+<pinref part="BAR_GRAPH" gate="A" pin="A"/>
+<wire x1="248.92" y1="30.48" x2="256.54" y2="30.48" width="0.1524" layer="91"/>
+</segment>
 </net>
 <net name="E" class="0">
@@
 </segment>
 <segment>
-<pinref part="BAR_GRAPH" gate="A" pin="A"/>
-<wire x1="248.92" y1="30.48" x2="256.54" y2="30.48" width="0.1524" layer="91"/>
-</segment>
-<segment>
-<pinref part="BAR_GRAPH" gate="F" pin="A"/>
-<wire x1="248.92" y1="15.24" x2="256.54" y2="15.24" width="0.1524" layer="91"/>
-</segment>
-</net>
+<pinref part="BAR_GRAPH" gate="J" pin="A"/>
+<wire x1="248.92" y1="5.08" x2="256.54" y2="5.08" width="0.1524" layer="91"/>
+</segment>
+<segment>
+<pinref part="BAR_GRAPH" gate="E" pin="A"/>
+<wire x1="248.92" y1="20.32" x2="256.54" y2="20.32" width="0.1524" layer="91"/>
+</segment>
+</net>
